File: MULTIIO/MULTIIO/CardSelect.kicad_sch (KiCad schematic)
At the start: 7 parts, among them SW1 BaseAddress, U1 74LS08, U2 74LS32, U7 74LS688, U8 74LS138, U9 74LS138

Commit message: multi io work
Connections:
- net VIA1_INT: no longer names the net of RN2.4 (R3)
- no-connect marks 10 -> 11
Changed lines of the file:
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@@
 	(title_block
 		(title "ISA MULTI IO ")
-		(date "2025-05-31")
-		(rev "v1")
+		(date "2025-07-19")
+		(rev "v1.1")
 		(company "DAN WERNER")
 	)
@@
 		(diameter 0)
 		(color 0 0 0 0)
+	)
+	(no_connect
+		(at 60.96 91.44)
 	)
 	(no_connect
@@
 		(pts
 			(xy 46.99 74.93) (xy 48.26 74.93)
-		)
-		(stroke
-			(width 0)
-			(type default)
-		)
-	)
-	(wire
-		(pts
-			(xy 60.96 88.9) (xy 60.96 91.44)
 		)
 		(stroke
@@
 				(hide yes)
 			)
-		)
-	)
-	(global_label "VIA1_INT"
-		(shape output)
-		(at 60.96 88.9 90)
-		(fields_autoplaced yes)
-		(effects
-			(font
-				(size 1.27 1.27)
-			)
-			(justify left)
-		)
-		(property "Intersheetrefs" "${INTERSHEET_REFS}"
-			(at 60.96 78.0528 90)
-			(effects
-				(font
-					(size 1.27 1.27)
-				)
-				(justify left)
-				(hide yes)
-			)
