File: MULTIIO/MULTIIO/IEC.kicad_sch (KiCad schematic)
At the start: 9 parts, among them J6 VIA INTERRUPT, J7 IEC PORT, U18 W65C22NxP, U2 74LS32, U3 7406

Commit message: multi io work
Parts:
- removed J6: VIA INTERRUPT, Custom:STD_DDW_PINHEAD_V_2x06, symbol Connector_Generic:Conn_02x06_Counter_Clockwise
- removed U18: W65C22NxP, Custom:STD_DDW_DIP40, symbol 65xx-library:W65C22NxP
- removed unit 5 of U3
- added U19: 74LS374, Custom:STD_DDW_DIP20, symbol 74xx:74LS374
- added U20: 74LS244, Custom:STD_DDW_DIP20, symbol 74xx:74LS244
- added U4: 74LS32, Custom:STD_DDW_DIP14, symbol 74xx:74LS32
Connections:
- net B_D0: now also U19.3 (D0), U20.18 (O0a)
- net B_D1: now also U19.4 (D1), U20.16 (O1a)
- net B_D2: now also U19.7 (D2), U20.14 (O2a)
- net B_D3: now also U19.8 (D3), U20.12 (O3a)
- net B_D4: now also U19.13 (D4), U20.9 (O0b)
- net B_D5: now also U19.14 (D5), U20.7 (O1b)
- net B_D6: now also U19.17 (D6), U20.5 (O2b)
- net B_D7: now also U19.18 (D7), U20.3 (O3b)
- net B_IOW: now also U4.5
- net CS_VIA1: now also U4.4, U4.9
- net GND: now also U19.1 (OE), U19.10 (GND), U20.10 (GND)
- net SERATNOUT: now also U19.2 (O0)
- net SERCLKIN: now also U20.2 (I0a)
- net SERCLKOUT: now also U19.5 (O1)
- net SERDATAIN: now also U20.4 (I1a)
- net SERDATAOUT: now also U19.6 (O2)
- net VCC: now also U19.20 (VCC), U20.20 (VCC)
- net SERSRQ: no longer names the net of J7.1
- new net: U19.11 (Cp), U4.6
- new net: U20.1 (OEa), U20.19 (OEb), U4.8
- new net B_IOR: U4.10
- no-connect marks 14 -> 12
