File: MULTIIO/MULTIIO/ISA.kicad_sch (KiCad schematic)
At the start: 1 part, among them J1 Bus_ISA_8bit_CUSTOM

Commit message: multi io work
Parts:
- added U5: 74LS06, Custom:STD_DDW_DIP14, symbol 74xx:74LS06
Connections:
- net ~{RESET}: now also U5.6; no longer J1.2 (RESET)
- new net RESET: J1.2 (RESET), U5.5
- no-connect marks 29 -> 30
Changed lines of the file:
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@@
 	(title_block
 		(title "ISA MULTI IO ")
-		(date "2025-05-31")
-		(rev "v1")
+		(date "2025-07-19")
+		(rev "v1.1")
 		(company "DAN WERNER")
 	)
@@
 	)
 	(no_connect
+		(at 52.07 88.9)
+	)
+	(no_connect
 		(at 87.63 63.5)
 	)
@@
 	(wire
 		(pts
+			(xy 59.69 144.78) (xy 62.23 144.78)
+		)
+		(stroke
+			(width 0)
+			(type default)
+		)
+	)
+	(wire
+		(pts
 			(xy 87.63 96.52) (xy 91.44 96.52)
 		)
@@
 		(pts
 			(xy 30.48 63.5) (xy 52.07 63.5)
+		)
+		(stroke
+			(width 0)
+			(type default)
+		)
+	)
+	(wire
+		(pts
+			(xy 77.47 144.78) (xy 81.28 144.78)
 		)
 		(stroke
@@
 		)
 	)
+	(global_label "~{RESET}"
+		(shape output)
+		(at 81.28 144.78 0)
+		(effects
+			(font
+				(size 1.27 1.27)
+			)
+			(justify left)
+		)
+		(property "Intersheetrefs" "${INTERSHEET_REFS}"
+			(at 81.28 144.78 0)
+			(effects
+				(font
+					(size 1.27 1.27)
+				)
+				(hide yes)
+			)
+		)
+	)
 	(global_label "IRQ3"
 		(shape output)
@@
 		)
 	)
+	(global_label "RESET"
+		(shape input)
+		(at 59.69 144.78 180)
+		(effects
+			(font
+				(size 1.27 1.27)
+			)
+			(justify right)
+		)
+		(property "Intersheetrefs" "${INTERSHEET_REFS}"
+			(at 59.69 144.78 0)
+			(effects
+				(font
+					(size 1.27 1.27)
+				)
+				(hide yes)
+			)
+		)
+	)
 	(global_label "B_A19"
 		(shape tri_state)
@@
 		)
 	)
-	(global_label "~{RESET}"
+	(global_label "RESET"
 		(shape input)
 		(at 49.53 43.18 180)
@@
 				)
 			)
+		)
+	)
+	(symbol
+		(lib_id "74xx:74LS06")
+		(at 69.85 144.78 0)
+		(unit 3)
+		(exclude_from_sim no)
+		(in_bom yes)
+		(on_board yes)
+		(dnp no)
+		(property "Reference" "U5"
+			(at 68.58 143.51 0)
+			(effects
+				(font
+					(size 1.27 1.27)
+				)
+			)
+		)
+		(property "Value" "74LS06"
+			(at 68.58 146.05 0)
+			(effects
+				(font
+					(size 1.27 1.27)
+				)
+			)
+		)
+		(property "Footprint" "Custom:STD_DDW_DIP14"
+			(at 69.85 144.78 0)
+			(effects
+				(font
+					(size 1.27 1.27)
+				)
+				(hide yes)
+			)
+		)
+		(property "Datasheet" "http://www.ti.com/lit/gpn/sn74LS06"
+			(at 69.85 144.78 0)
+			(effects
+				(font
+					(size 1.27 1.27)
+				)
+				(hide yes)
+			)
+		)
+		(property "Description" ""
+			(at 69.85 144.78 0)
+			(effects
+				(font
+					(size 1.27 1.27)
+				)
+				(hide yes)
+			)
+		)
+		(pin "1"
+		)
+		(pin "2"
+		)
+		(pin "3"
+		)
+		(pin "4"
+		)
+		(pin "5"
+		)
+		(pin "6"
+		)
+		(pin "8"
+		)
+		(pin "9"
+		)
+		(pin "10"
+		)
+		(pin "11"
+		)
+		(pin "12"
+		)
+		(pin "13"
+		)
+		(pin "14"
+		)
+		(pin "7"
+		)
+		(instances
+			(project "MULTIIO"
+				(path "/8d0f25e7-72aa-42f1-b96d-60e778d112e0/2e54f558-6be6-45f0-89e1-ea204c8ee7c2"
+					(reference "U5")
+					(unit 3)
+				)
+			)
