File: MULTIIO/MULTIIO/MULTIIO.kicad_pcb (KiCad board)
At the start: 2 copper layers, 176.7 x 111.9 mm, 79 parts, among them J1 Bus_ISA_8bit_CUSTOM, J2 KM INTERRUPT, J3 MOUSE, J4 KEYBOARD, J5 PAR INTERRUPT, J6 VIA INTERRUPT, J7 IEC PORT, P1 PARALLEL, SW1 BaseAddress, U1 74LS08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

Commit message: multi io work
Parts:
- removed J6: VIA INTERRUPT, Custom:STD_DDW_PINHEAD_V_2x06
- removed U18: W65C22NxP, Custom:STD_DDW_DIP40
- added U19: 74LS374, Custom:STD_DDW_DIP20, F.Cu at (289.6, 95.6)
- added U20: 74LS244, Custom:STD_DDW_DIP20, F.Cu at (278.1, 69.2)
- moved U1 153.4 mm to (302.5, 100.2)
- moved U12 145.3 mm to (302.8, 78.1)
- moved C10 96.2 mm to (313.7, 104.9)
- moved U9 85.3 mm to (155.7, 53.7)
- moved U16 25.8 mm to (237.5, 87.2)
- moved C14 18.1 mm to (237.2, 68.6), turned to 0 degrees
- moved SW1 17.5 mm to (221.5, 84.4)
- moved C16 5.63 mm to (289.3, 57.9)
Connections:
- J1 pad 2: ~{RESET} -> RESET
- J7 pad 1: SERSRQ -> unconnected-(J7-Pad1)
- RN2 pad 4: VIA1_INT -> unconnected-(RN2-R3-Pad4)
- RN4 pad 7: unconnected-(RN4-R6-Pad7) -> ~{RESET}
- U3 pad 10: Net-(J6-Pin_1) -> unconnected-(U3-Pad10)
- U3 pad 11: VIA1_INT -> unconnected-(U3-Pad11)
- U4 pad 10: unconnected-(U4-Pad10) -> B_IOR
- U4 pad 4: unconnected-(U4-Pad4) -> CS_VIA1
- U4 pad 5: unconnected-(U4-Pad5) -> B_IOW
- U4 pad 6: unconnected-(U4-Pad6) -> Net-(U19-Cp)
- U4 pad 8: unconnected-(U4-Pad8) -> Net-(U20-OEa)
- U4 pad 9: unconnected-(U4-Pad9) -> CS_VIA1
- U5 pad 5: unconnected-(U5-Pad5) -> RESET
- U5 pad 6: unconnected-(U5-Pad6) -> ~{RESET}
Routing:
- net RESET: track 0.00 -> 200.3 mm, vias 0 -> 4
- net 470D: track 202.7 -> 38.9 mm
- net Net-(U19-Cp): track 0.00 -> 154.3 mm, vias 0 -> 3
- net VIA1_INT: track 130.5 -> 0.00 mm, vias 1 -> 0
- net Net-(U7-G): track 190.3 -> 65.9 mm, vias 2 -> 1
- net Net-(U20-OEa): track 0.00 -> 117.6 mm, vias 0 -> 2
- net Net-(U11-P23): track 160.5 -> 45.8 mm, vias 3 -> 1
- net Net-(U11-P22): track 163.0 -> 54.8 mm, vias 3 -> 1
- net CS_VIA1: track 170.8 -> 65.3 mm, vias 2 -> 0
- net Net-(J6-Pin_1): track 100.8 -> 0.00 mm, vias 1 -> 0
- net SERSRQ: track 94.5 -> 0.00 mm, vias 1 -> 0
- net Net-(U11-P26/DRQ): track 132.0 -> 40.2 mm, vias 2 -> 1
- net GND: track 858.7 -> 947.0 mm
- net Net-(U11-P27/DAK): track 122.9 -> 42.3 mm, vias 1 -> 0
- net B_CLK: track 79.6 -> 0.00 mm, vias 2 -> 0
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Other:
- board text added: "ISA MultiIO Dan Werner V1.1 7/19/2025"
- board text removed: "ISA MultiIO Dan Werner V1 6/8/2025"
