File: MULTIIO/MULTIIO/MULTIIO.kicad_sch (KiCad schematic)
At the start: 28 parts, among them U1 74LS08, U12 74LS06, U2 74LS32, U3 7406, U4 74LS32, U5 74LS06, U6 74LS04

Commit message: multi io work
Parts:
- removed unit 2 of U4
- removed unit 3 of U4
- removed unit 3 of U5
- added unit 5 of U3
Connections:
- no-connect marks 22 -> 16
Changed lines of the file:
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@@
 	(title_block
 		(title "ISA MULTI IO ")
-		(date "2025-05-31")
-		(rev "v1")
+		(date "2025-07-19")
+		(rev "v1.1")
 		(company "DAN WERNER")
 	)
@@
 	)
 	(no_connect
+		(at 41.91 182.88)
+	)
+	(no_connect
 		(at 21.59 167.64)
 	)
 	(no_connect
-		(at 64.77 168.91)
+		(at 57.15 182.88)
 	)
 	(no_connect
@@
 	)
 	(no_connect
-		(at 63.5 182.88)
-	)
-	(no_connect
 		(at 41.91 153.67)
 	)
 	(no_connect
-		(at 48.26 182.88)
-	)
-	(no_connect
 		(at 60.96 127)
 	)
 	(no_connect
-		(at 64.77 177.8)
-	)
-	(no_connect
 		(at 20.32 180.34)
 	)
@@
 	)
 	(no_connect
-		(at 64.77 182.88)
-	)
-	(no_connect
-		(at 80.01 166.37)
-	)
-	(no_connect
-		(at 80.01 180.34)
-	)
-	(no_connect
 		(at 80.01 151.13)
 	)
 	(no_connect
-		(at 64.77 163.83)
-	)
-	(no_connect
 		(at 64.77 148.59)
 	)
@@
 	(symbol
 		(lib_id "74xx:74LS06N")
+		(at 49.53 182.88 0)
+		(unit 5)
+		(exclude_from_sim no)
+		(in_bom yes)
+		(on_board yes)
+		(dnp no)
+		(property "Reference" "U3"
+			(at 52.07 180.34 0)
+			(effects
+				(font
+					(size 1.27 1.27)
+				)
+			)
+		)
+		(property "Value" "7406"
+			(at 48.26 182.88 0)
+			(effects
+				(font
+					(size 1.27 1.27)
+				)
+			)
+		)
+		(property "Footprint" "Custom:STD_DDW_DIP14"
+			(at 49.53 182.88 0)
+			(effects
+				(font
+					(size 1.27 1.27)
+				)
+				(hide yes)
+			)
+		)
+		(property "Datasheet" "http://www.ti.com/lit/gpn/sn74LS06N"
+			(at 49.53 182.88 0)
+			(effects
+				(font
+					(size 1.27 1.27)
+				)
+				(hide yes)
+			)
+		)
+		(property "Description" ""
+			(at 49.53 182.88 0)
+			(effects
+				(font
+					(size 1.27 1.27)
+				)
+				(hide yes)
+			)
+		)
+		(pin "1"
+		)
+		(pin "2"
+		)
+		(pin "3"
+		)
+		(pin "4"
+		)
+		(pin "5"
+		)
+		(pin "6"
+		)
+		(pin "8"
+		)
+		(pin "9"
+		)
+		(pin "10"
+		)
+		(pin "11"
+		)
+		(pin "12"
+		)
+		(pin "13"
+		)
+		(pin "14"
+		)
+		(pin "7"
+		)
+		(instances
+			(project "MULTIIO"
+				(path "/8d0f25e7-72aa-42f1-b96d-60e778d112e0"
+					(reference "U3")
+					(unit 5)
+				)
+			)
+		)
+	)
+	(symbol
+		(lib_id "74xx:74LS06N")
 		(at 49.53 165.1 0)
 		(unit 4)
@@
 	)
 	(symbol
-		(lib_id "74xx:74LS32")
-		(at 72.39 166.37 0)
-		(unit 2)
-		(exclude_from_sim no)
-		(in_bom yes)
-		(on_board yes)
-		(dnp no)
-		(fields_autoplaced yes)
-		(property "Reference" "U4"
-			(at 72.39 157.48 0)
-			(effects
-				(font
-					(size 1.27 1.27)
-				)
-			)
-		)
-		(property "Value" "74LS32"
-			(at 72.39 160.02 0)
-			(effects
-				(font
-					(size 1.27 1.27)
-				)
-			)
-		)
-		(property "Footprint" "Custom:STD_DDW_DIP14"
-			(at 72.39 166.37 0)
-			(effects
-				(font
-					(size 1.27 1.27)
-				)
-				(hide yes)
-			)
-		)
-		(property "Datasheet" "http://www.ti.com/lit/gpn/sn74LS32"
-			(at 72.39 166.37 0)
-			(effects
-				(font
-					(size 1.27 1.27)
-				)
-				(hide yes)
-			)
-		)
-		(property "Description" "Quad 2-input OR"
-			(at 72.39 166.37 0)
-			(effects
-				(font
-					(size 1.27 1.27)
-				)
-				(hide yes)
-			)
-		)
-		(pin "13"
-		)
-		(pin "8"
-		)
-		(pin "4"
-		)
-		(pin "9"
-		)
-		(pin "10"
-		)
-		(pin "12"
-		)
-		(pin "1"
-		)
-		(pin "14"
-		)
-		(pin "11"
-		)
-		(pin "5"
-		)
-		(pin "7"
-		)
-		(pin "2"
-		)
-		(pin "6"
-		)
-		(pin "3"
-		)
-		(instances
-			(project ""
-				(path "/8d0f25e7-72aa-42f1-b96d-60e778d112e0"
-					(reference "U4")
-					(unit 2)
-				)
-			)
-		)
-	)
-	(symbol
 		(lib_id "power:VCC")
 		(at 93.98 138.43 0)
@@
 	)
 	(symbol
-		(lib_id "74xx:74LS06")
-		(at 55.88 182.88 0)
-		(unit 3)
-		(exclude_from_sim no)
-		(in_bom yes)
-		(on_board yes)
-		(dnp no)
-		(property "Reference" "U5"
-			(at 54.61 181.61 0)
-			(effects
-				(font
-					(size 1.27 1.27)
-				)
-			)
-		)
-		(property "Value" "74LS06"
-			(at 54.61 184.15 0)
-			(effects
-				(font
-					(size 1.27 1.27)
-				)
-			)
-		)
-		(property "Footprint" "Custom:STD_DDW_DIP14"
-			(at 55.88 182.88 0)
-			(effects
-				(font
-					(size 1.27 1.27)
-				)
-				(hide yes)
-			)
-		)
-		(property "Datasheet" "http://www.ti.com/lit/gpn/sn74LS06"
-			(at 55.88 182.88 0)
-			(effects
-				(font
-					(size 1.27 1.27)
-				)
-				(hide yes)
-			)
-		)
-		(property "Description" ""
-			(at 55.88 182.88 0)
-			(effects
-				(font
-					(size 1.27 1.27)
-				)
-				(hide yes)
-			)
-		)
-		(pin "1"
-		)
-		(pin "2"
-		)
-		(pin "3"
-		)
-		(pin "4"
-		)
-		(pin "5"
-		)
-		(pin "6"
-		)
-		(pin "8"
-		)
-		(pin "9"
-		)
-		(pin "10"
-		)
-		(pin "11"
-		)
-		(pin "12"
-		)
-		(pin "13"
-		)
-		(pin "14"
-		)
-		(pin "7"
-		)
-		(instances
-			(project "MULTIIO"
-				(path "/8d0f25e7-72aa-42f1-b96d-60e778d112e0"
-					(reference "U5")
-					(unit 3)
-				)
-			)
-		)
-	)
-	(symbol
 		(lib_id "Device:C")
 		(at 170.18 116.84 0)
@@
 				)
 			)
-		)
-	)
-	(symbol
-		(lib_id "74xx:74LS32")
-		(at 72.39 180.34 0)
-		(unit 3)
-		(exclude_from_sim no)
-		(in_bom yes)
-		(on_board yes)
-		(dnp no)
-		(fields_autoplaced yes)
-		(property "Reference" "U4"
-			(at 72.39 171.45 0)
-			(effects
-				(font
-					(size 1.27 1.27)
-				)
-			)
-		)
-		(property "Value" "74LS32"
-			(at 72.39 173.99 0)
-			(effects
-				(font
-					(size 1.27 1.27)
-				)
-			)
-		)
-		(property "Footprint" "Custom:STD_DDW_DIP14"
-			(at 72.39 180.34 0)
-			(effects
-				(font
-					(size 1.27 1.27)
-				)
-				(hide yes)
-			)
-		)
-		(property "Datasheet" "http://www.ti.com/lit/gpn/sn74LS32"
-			(at 72.39 180.34 0)
-			(effects
-				(font
-					(size 1.27 1.27)
-				)
-				(hide yes)
-			)
-		)
-		(property "Description" "Quad 2-input OR"
-			(at 72.39 180.34 0)
-			(effects
-				(font
-					(size 1.27 1.27)
-				)
-				(hide yes)
-			)
-		)
-		(pin "13"
-		)
-		(pin "8"
-		)
-		(pin "4"
-		)
-		(pin "9"
-		)
-		(pin "10"
-		)
-		(pin "12"
-		)
-		(pin "1"
-		)
-		(pin "14"
-		)
-		(pin "11"
-		)
-		(pin "5"
-		)
-		(pin "7"
-		)
-		(pin "2"
-		)
-		(pin "6"
-		)
-		(pin "3"
-		)
-		(instances
-			(project ""
-				(path "/8d0f25e7-72aa-42f1-b96d-60e778d112e0"
-					(reference "U4")
-					(unit 3)
-				)
-			)
