File: MULTIIO/MULTIIO/Printer.kicad_sch (KiCad schematic)
At the start: 33 parts, among them J5 PAR INTERRUPT, P1 PARALLEL, U13 74LS374, U14 74LS374, U15 74LS244, U16 74LS244, U17 74LS244, U2 74LS32, U5 74LS06, U6 74LS04

Commit message: multi io work
Connections:
- net ~{RESET}: now reaches RN4.7 (R6)
- no-connect marks 3 -> 2
Changed lines of the file:
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@@
 	(title_block
 		(title "ISA MULTI IO ")
-		(date "2025-05-31")
-		(rev "v1")
+		(date "2025-07-19")
+		(rev "v1.1")
 		(company "DAN WERNER")
 	)
@@
 		(at 284.48 241.3)
 	)
-	(no_connect
-		(at 284.48 236.22)
-	)
 	(wire
 		(pts
@@
 	(wire
 		(pts
+			(xy 284.48 236.22) (xy 295.91 236.22)
+		)
+		(stroke
+			(width 0)
+			(type default)
+		)
+	)
+	(wire
+		(pts
 			(xy 50.8 134.62) (xy 39.37 134.62)
 		)
@@
 				(hide yes)
 			)
+		)
+	)
+	(global_label "~{RESET}"
+		(shape input)
+		(at 295.91 236.22 0)
+		(effects
+			(font
+				(size 1.27 1.27)
+			)
+			(justify left)
+		)
+		(property "Intersheetrefs" "${INTERSHEET_REFS}"
+			(at 295.91 236.22 0)
+			(effects
+				(font
+					(size 1.27 1.27)
+				)
+				(hide yes)
+			)
