File: DUALESP/HARDWARE/DUALESP.kicad_sch (KiCad schematic)
At the start: 22 parts, among them U17 74LS08, U4 74LS04, U5 74LS32, U6 74LS07, U7 74LS32, U8 74LS32

Commit message: ESPIO updates
Changed lines of the file:
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@@
 (kicad_sch
-	(version 20231120)
+	(version 20250114)
 	(generator "eeschema")
-	(generator_version "8.0")
+	(generator_version "9.0")
 	(paper "USLedger")
 	(title_block
 		(title "ISA DUAL ESP32")
-		(date "2025-06-21")
-		(rev "V1.1")
+		(date "2025-06-28")
+		(rev "V1.2")
 	)
 	(junction
@@
 		(at 35.052 25.4)
 		(size 86.614 50.8)
+		(exclude_from_sim no)
+		(in_bom yes)
+		(on_board yes)
+		(dnp no)
 		(fields_autoplaced yes)
 		(stroke
@@
 		(at 239.522 22.606)
 		(size 75.184 53.086)
+		(exclude_from_sim no)
+		(in_bom yes)
+		(on_board yes)
+		(dnp no)
 		(fields_autoplaced yes)
 		(stroke
@@
 		(at 136.144 24.13)
 		(size 79.248 53.086)
+		(exclude_from_sim no)
+		(in_bom yes)
+		(on_board yes)
+		(dnp no)
 		(fields_autoplaced yes)
 		(stroke
@@
 		)
 	)
+	(embedded_fonts no)
 )

Commit message: ESPIO updates
Parts:
- removed D1: LED, Custom:STD_DDW_LED5, symbol Device:LED
- removed R1: 470Ω, Custom:STD_DDW_RESISTOR, symbol Device:R
- added unit 3 of U6
- added unit 2 of U6
- added unit 1 of U6
- added unit 4 of U6
- U5, U7, U8: value 74LS32 -> 74F32
Connections:
- no-connect marks 21 -> 29
