File: VIDEO/HARDWARE/CardSelect.kicad_sch (KiCad schematic)
At the start: 13 parts, among them SW1 BaseAddress, SW2 Memory Window, U18 74LS244, U2 74LS32, U3 74LS08, U4 74LS244, U40 SRAM-32K, U5 74LS244, U6 74LS245, U7 74LS688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

Commit message: sound updates
Parts:
- removed RN2: 4.7k, Custom:STD_DDW_SIP9, symbol Device:R_Network08
- removed SW1: BaseAddress, Custom:STD_DDW_DIP10, symbol Switch:SW_DIP_x05
- removed U3: 74LS08, Custom:STD_DDW_DIP14, symbol 74xx:74LS08
- removed U7: 74LS688, Custom:STD_DDW_DIP20, symbol 74xx:74LS688
Connections:
- no-connect marks 8 -> 5
Other:
- title: ISA VIDEO/SID -> ISA VIDEO
