File: VIDEO/HARDWARE/ISA.kicad_sch (KiCad schematic)
At the start: 1 part, among them J6 Bus_ISA_8bit_CUSTOM

Commit message: sound updates
Connections:
- net B_IOR: no longer names the net of J6.14 (~{IOR})
- net B_IOW: no longer names the net of J6.13 (~{IOW})
- net ~{RESET}: no longer names the net of J6.2 (RESET)
- no-connect marks 22 -> 25
Other:
- title: ISA VIDEO/SID -> ISA VIDEO
Changed lines of the file:
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@@
 	(paper "A4")
 	(title_block
-		(title "ISA VIDEO/SID")
-		(date "2026-01-31")
-		(rev "V1.1")
+		(title "ISA VIDEO")
+		(date "2026-03-22")
+		(rev "V1.6")
 	)
 	(junction
@@
 	)
 	(no_connect
+		(at 59.69 67.31)
+	)
+	(no_connect
 		(at 59.69 80.01)
 	)
@@
 	)
 	(no_connect
+		(at 59.69 64.77)
+	)
+	(no_connect
 		(at 59.69 69.85)
 	)
@@
 	)
 	(no_connect
+		(at 59.69 36.83)
+	)
+	(no_connect
 		(at 59.69 77.47)
 	)
@@
 	(wire
 		(pts
-			(xy 57.15 36.83) (xy 59.69 36.83)
-		)
-		(stroke
-			(width 0)
-			(type default)
-		)
-	)
-	(wire
-		(pts
 			(xy 95.25 54.61) (xy 99.06 54.61)
 		)
@@
 	(wire
 		(pts
-			(xy 54.61 64.77) (xy 59.69 64.77)
-		)
-		(stroke
-			(width 0)
-			(type default)
-		)
-	)
-	(wire
-		(pts
 			(xy 95.25 52.07) (xy 99.06 52.07)
 		)
@@
 	(wire
 		(pts
+			(xy 59.69 92.71) (xy 55.88 92.71)
+		)
+		(stroke
+			(width 0)
+			(type default)
+		)
+	)
+	(wire
+		(pts
+			(xy 59.69 85.09) (xy 55.88 85.09)
+		)
+		(stroke
+			(width 0)
+			(type default)
+		)
+	)
+	(wire
+		(pts
+			(xy 95.25 41.91) (xy 99.06 41.91)
+		)
+		(stroke
+			(width 0)
+			(type default)
+		)
+	)
+	(wire
+		(pts
 			(xy 41.91 34.29) (xy 59.69 34.29)
 		)
@@
 	(wire
 		(pts
-			(xy 59.69 92.71) (xy 55.88 92.71)
-		)
-		(stroke
-			(width 0)
-			(type default)
-		)
-	)
-	(wire
-		(pts
-			(xy 59.69 85.09) (xy 55.88 85.09)
-		)
-		(stroke
-			(width 0)
-			(type default)
-		)
-	)
-	(wire
-		(pts
-			(xy 95.25 41.91) (xy 99.06 41.91)
-		)
-		(stroke
-			(width 0)
-			(type default)
-		)
-	)
-	(wire
-		(pts
 			(xy 95.25 77.47) (xy 99.06 77.47)
 		)
@@
 		(pts
 			(xy 95.25 90.17) (xy 99.06 90.17)
-		)
-		(stroke
-			(width 0)
-			(type default)
-		)
-	)
-	(wire
-		(pts
-			(xy 54.61 67.31) (xy 59.69 67.31)
 		)
 		(stroke
@@
 		)
 	)
-	(global_label "~{RESET}"
-		(shape input)
-		(at 57.15 36.83 180)
-		(effects
-			(font
-				(size 1.27 1.27)
-			)
-			(justify right)
-		)
-		(property "Intersheetrefs" "${INTERSHEET_REFS}"
-			(at 57.15 36.83 0)
-			(effects
-				(font
-					(size 1.27 1.27)
-				)
-				(hide yes)
-			)
-		)
-	)
 	(global_label "TC"
 		(shape input)
@@
 		)
 	)
-	(global_label "B_IOW"
-		(shape input)
-		(at 54.61 64.77 180)
-		(fields_autoplaced yes)
-		(effects
-			(font
-				(size 1.27 1.27)
-			)
-			(justify right)
-		)
-		(property "Intersheetrefs" "${INTERSHEET_REFS}"
-			(at 46.0005 64.77 0)
-			(effects
-				(font
-					(size 1.27 1.27)
-				)
-				(justify right)
-				(hide yes)
-			)
-		)
-	)
 	(global_label "B_A12"
 		(shape tri_state)
@@
 				(hide yes)
 			)
-		)
-	)
-	(global_label "B_IOR"
-		(shape input)
-		(at 54.61 67.31 180)
-		(fields_autoplaced yes)
-		(effects
-			(font
-				(size 1.27 1.27)
-			)
-			(justify right)
-		)
-		(property "Intersheetrefs" "${INTERSHEET_REFS}"
-			(at 46.1819 67.31 0)
-			(effects
-				(font
-					(size 1.27 1.27)
-				)
-				(justify right)
-				(hide yes)
-			)
