File: VIDEO/HARDWARE/esp.kicad_sch (KiCad schematic)
At the start: 20 parts, among them J11 DE15_Receptacle_HighDensity, U1 LP2950-3.3_TO92, U32 74LVC245, U33 74LVC245, U34 74LVC245, U36 Pico

Commit message: version 1.1
Parts:
- removed R1, R3: 1KΩ, Custom:STD_DDW_RESISTOR, symbol Device:R_Small
- added U8: 74LVC245, Custom:STD_DDW_DIP20, symbol 74xx:74LS245
Connections:
- net +3.3V: now also U8.20 (VCC)
- net CLK_CPU: now also U8.17 (B1)
- net GND: now also U8.1 (A->B), U8.10 (GND), U8.19 (CE)
- net MEMW: now also U8.18 (B0)
- net V_CLK: now also U8.3 (A1)
- net V_RW: now also U8.2 (A0)
- no-connect marks 19 -> 31

Commit message: sound updates
Other:
- title: ISA VIDEO/SID -> ISA VIDEO
Changed lines of the file:
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@@
 	(paper "USLedger")
 	(title_block
-		(title "ISA VIDEO/SID")
-		(date "2026-01-31")
-		(rev "V1.1")
+		(title "ISA VIDEO")
+		(date "2026-03-22")
+		(rev "V1.6")
 	)
 	(junction
