File: VIDEO/HARDWARE/video.kicad_pcb (KiCad board)
At the start: 2 copper layers, 176.7 x 111.9 mm, 63 parts, among them J11 DE15_Receptacle_HighDensity, J24 SID OUT, J6 Bus_ISA_8bit_CUSTOM, P3 1 MHz CLK, SW1 BaseAddress, SW2 Memory Window, U1 LP2950-3.3_TO92, U16 6581, U18 74LS244, U19 74LS374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

Commit message: version 1.1
Parts:
- removed R1, R3: 1KΩ, Custom:STD_DDW_RESISTOR
- added C15: 0.1µF, Custom:STD_DDW_CAP, F.Cu at (74.9, 101.4)
- added C16: 0.1µF, Custom:STD_DDW_CAP, F.Cu at (58.9, 101.4)
- added C17: 0.1µF, Custom:STD_DDW_CAP, F.Cu at (44.2, 100.0)
- added C18: 0.1µF, Custom:STD_DDW_CAP, F.Cu at (82.8, 67.8)
- added U8: 74LVC245, Custom:STD_DDW_DIP20, F.Cu at (85.0, 84.9)
- moved C11 101.9 mm to (159.6, 82.5)
- moved C2 81.6 mm to (115.1, 57.8)
- moved J24 58.7 mm to (215.1, 106.2)
- moved C1 36.0 mm to (92.0, 69.1)
- moved U1 19.9 mm to (84.6, 50.7)
- moved U5 0.18 mm to (99.3, 85.0)
Routing:
- net V_RW: track 157.1 -> 28.8 mm
- net V_CLK: track 145.6 -> 17.4 mm
- net VGAB2K: track 161.1 -> 235.9 mm, vias 0 -> 6
- net VGAG2K: track 137.8 -> 210.3 mm
- net VGAG1L: track 126.4 -> 196.5 mm, vias 0 -> 1
- net CLK_CPU: track 127.6 -> 69.0 mm, vias 2 -> 3
- net VGAR2K: track 183.0 -> 125.7 mm, vias 2 -> 0
- net B_A3: track 208.9 -> 263.2 mm, vias 5 -> 2
- net B_A4: track 184.9 -> 236.3 mm
- net VIDEO_WINDOW: track 289.4 -> 239.2 mm, vias 11 -> 4
- net Net-(J24-Ext): track 40.4 -> 90.4 mm, vias 0 -> 1
- net VGAR1K: track 181.1 -> 133.5 mm, vias 2 -> 0
- net bA11: track 148.5 -> 107.4 mm, vias 6 -> 1
- net bA5: track 148.6 -> 108.8 mm, vias 6 -> 1
- net VSYNC: track 221.7 -> 186.5 mm, vias 3 -> 1
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Other:
- board text added: "ISA VIDEO/SID Dan Werner V1.1 1/31/2026"
- board text removed: "ISA VIDEO/SID Dan Werner V1.0 1/18/2026"

Commit message: sound updates
Parts:
- removed C37: 0.1 uF, Custom:STD_DDW_CAP
- removed C38: 0.22uf, Custom:STD_DDW_PCAP
- removed C39, C43: 10uf, Custom:STD_DDW_PCAP
- removed C42, C46: 2200pf, Custom:STD_DDW_CAP
- removed C44, C45: 470pf, Custom:STD_DDW_CAP
- removed C50: 0.47uf, Custom:STD_DDW_PCAP
- removed J24: SID OUT, Custom:CUI_RCJ-047
- removed JP3: SID CS, Custom:STD_DDW_PINHEAD_V_1x03
- removed P3: 1 MHz CLK, Custom:STD_DDW_DIP14
- removed RN2: 4.7k, Custom:STD_DDW_SIP9
- removed SW1: BaseAddress, Custom:STD_DDW_DIP10
- removed U16: 6581, Custom:STD_DDW_DIP28
- removed U19, U20: 74LS374, Custom:STD_DDW_DIP20
- removed U3: 74LS08, Custom:STD_DDW_DIP14
- removed U7: 74LS688, Custom:STD_DDW_DIP20
- moved C3 51.3 mm to (170.1, 71.9)
- moved C7 20.2 mm to (152.7, 42.0)
Connections:
- J6 pad 13: B_IOW -> unconnected-(J6-~{IOW}-Pad13)
- J6 pad 14: B_IOR -> unconnected-(J6-~{IOR}-Pad14)
- J6 pad 2: ~{RESET} -> unconnected-(J6-RESET-Pad2)
Routing:
- net B_A3: track 263.2 -> 59.8 mm, vias 2 -> 0
- net B_A4: track 236.3 -> 50.1 mm, vias 3 -> 0
- net B_A6: track 243.3 -> 61.4 mm, vias 4 -> 1
- net B_A5: track 227.4 -> 53.5 mm, vias 6 -> 0
- net +12V: track 155.0 -> 0.00 mm
- net B_A7: track 222.4 -> 70.6 mm
- net GND: track 1011.1 -> 863.3 mm
- net B_A2: track 206.5 -> 64.4 mm, vias 5 -> 0
- net ~{SIDSEL}: track 141.0 -> 0.00 mm, vias 5 -> 0
- net Net-(U7-G): track 140.6 -> 0.00 mm
- net B_A0: track 200.0 -> 67.1 mm, vias 5 -> 0
- net B_A1: track 195.9 -> 65.1 mm, vias 3 -> 0
- net ~{RESET}: track 121.6 -> 0.00 mm, vias 4 -> 0
- net Net-(J24-Ext): track 90.4 -> 0.00 mm, vias 1 -> 0
- net SIDCLK: track 87.0 -> 0.00 mm, vias 1 -> 0
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Other:
- board text added: "ISA VIDEO Dan Werner V1.6 3/22/2026"
- board text removed: "ISA VIDEO/SID Dan Werner V1.1 1/31/2026"
