File: VIDEO/HARDWARE/video.kicad_sch (KiCad schematic)
At the start: 16 parts, among them U2 74LS32, U3 74LS08

Commit message: version 1.1
Parts:
- added C15, C16, C17, C18: 0.1µF, Custom:STD_DDW_CAP, symbol Device:C
Connections:
- net GND: now also C15.2, C16.2, C17.2, C18.2
- new net +3.3V: C15.1, C16.1, C17.1, C18.1

Commit message: sound updates
Parts:
- removed U3: 74LS08, Custom:STD_DDW_DIP14, symbol 74xx:74LS08
Connections:
- no-connect marks 18 -> 9
Other:
- removed sheet audio
- title: ISA VIDEO/SID -> ISA VIDEO
