File: SOUND/CardSelect.kicad_sch (KiCad schematic)
At the start: 9 parts, among them J2 Conn_02x06_Odd_Even, SW2 BaseAddress, U1 74LS08, U4 74LS244, U5 74LS06, U6 74LS245, U7 74LS688

Commit message: sound card working
Parts:
- removed NT1: NetTie_2, NetTie:NetTie-2_THT_Pad1.0mm, symbol Device:NetTie_2
- added U3: 74LS32, Custom:STD_DDW_DIP14, symbol 74xx:74LS32
Connections:
- net BoardSelect: now also U3.9
- net IOR: now also U3.10; no longer U6.1 (A->B)
- net A2: no longer names the net of U4.14 (O2a)
- net A3: no longer names the net of U4.12 (O3a)
- net B_A2: no longer names the net of U4.6 (I2a)
- net B_A3: no longer names the net of U4.8 (I3a)
- new net: U3.8, U6.1 (A->B)
- no-connect marks 6 -> 10
