File: SOUND/ISA.kicad_sch (KiCad schematic)
At the start: 2 parts, among them J1 Bus_ISA_8bit_CUSTOM, U5 74LS06

Commit message: sound card working
Parts:
- added R1: 1KΩ, Custom:STD_DDW_RESISTOR, symbol Device:R_Small
Connections:
- net GND: now also R1.2
- net RESET: now also R1.1
- no-connect marks 29 -> 31
