File: SOUND/SOUND.kicad_pcb (KiCad board)
At the start: 2 copper layers, 176.7 x 111.9 mm, 44 parts, among them J1 Bus_ISA_8bit_CUSTOM, J10 DB9_Male, J2 Conn_02x06_Odd_Even, J8 AudioJack3, J9 DB9_Male, P2 CHAN_MIX, SW2 BaseAddress, U1 74LS08, U2 W65C22NxP, U25 AY-3-8910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

Commit message: sound card working
Parts:
- removed NT1: NetTie_2, NetTie:NetTie-2_THT_Pad1.0mm
- removed U2: W65C22NxP, Custom:STD_DDW_DIP40
- added R1: 1KΩ, Custom:STD_DDW_RESISTOR, F.Cu at (276.6, 113.1)
- added U3: 74LS32, Custom:STD_DDW_DIP14, F.Cu at (201.2, 88.4)
- added U8: 8255, Custom:STD_DDW_DIP40, F.Cu at (221.0, 67.5)
- J10, J9: footprint Connector_Dsub:DSUB-9_Pins_Horizontal_P2.77x2.54mm_EdgePinOffset9.40mm -> Connector_Dsub:DSUB-9_Pins_Horizontal_P2.77x2.84mm_EdgePinOffset4.94mm_Housed_MountingHolesOffset4.94mm
- J8: footprint Connector_Audio:Jack_3.5mm_CUI_SJ1-3533NG_Horizontal_CircularHoles -> Custom:ddw_Jack_3.5mm_CUI_SJ1-3525N_Horizontal
- R10, R11, R12, R13, R14, R8, R9: footprint Resistor_THT:R_Axial_DIN0204_L3.6mm_D1.6mm_P5.08mm_Horizontal -> Custom:STD_DDW_RESISTOR
- moved C2 19.5 mm to (201.7, 73.6)
- moved C45 16.2 mm to (300.9, 94.9)
- moved R9 13.4 mm to (274.1, 66.3), turned to 0 degrees
- moved R12 13.2 mm to (273.8, 96.0)
- moved C44 10.9 mm to (300.3, 67.9)
- moved J8 8.44 mm to (320.4, 88.7)
- moved J9 4.26 mm to (317.0, 70.0)
- moved J10 4.16 mm to (317.0, 118.3)
- moved RN1 3.23 mm to (296.0, 54.0)
- moved C18 2.86 mm to (311.3, 45.6)
- moved R8 1.41 mm to (274.2, 59.6), turned to 0 degrees
Connections:
- J8 pad R: Net-(C47-Pad2) -> Net-(C46-Pad2)
- J8 pad S: Net-(C46-Pad2) -> GND
- J8 pad T: GND -> Net-(C47-Pad2)
- U25 pad 23: RESET -> ~{RESET}
- U4 pad 12: A3 -> unconnected-(U4-O3a-Pad12)
- U4 pad 14: A2 -> unconnected-(U4-O2a-Pad14)
- U4 pad 6: B_A2 -> unconnected-(U4-I2a-Pad6)
- U4 pad 8: B_A3 -> unconnected-(U4-I3a-Pad8)
- U6 pad 1: IOR -> Net-(U6-A->B)
Routing:
- net A3: track 75.0 -> 0.00 mm
- net A2: track 72.5 -> 0.00 mm
- net IOR: track 24.6 -> 81.7 mm
- net IOW: track 46.3 -> 92.8 mm, vias 1 -> 0
- net B_CLK: track 105.8 -> 61.8 mm
- net RESET: track 122.6 -> 162.3 mm, vias 0 -> 1
- net B_A2: track 39.5 -> 0.00 mm, vias 1 -> 0
- net B_A3: track 36.0 -> 0.00 mm, vias 1 -> 0
- net USERB_1: track 57.0 -> 87.4 mm
- net Net-(U6-A->B): track 0.00 -> 30.2 mm
- net ~{IRQ}: track 97.8 -> 68.8 mm, vias 1 -> 0
- net USERB_0: track 57.0 -> 84.3 mm
- net GND: track 701.3 -> 723.2 mm
- net P2_D: track 111.7 -> 133.3 mm
- net Net-(P2-Pin_1): track 45.7 -> 67.3 mm
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Other:
- board text added: "IO ADDRESS"
- board text added: "ISA SOUND Dan Werner V0.96 5/29/2026"
- board text added: "X"
- board text removed: "ISA SOUND Dan Werner V1.1 7/19/2025"
