File: SOUND/SOUND.kicad_sch (KiCad schematic)
At the start: 15 parts, among them U1 74LS08, U5 74LS06

Commit message: sound card working
Parts:
- added U3: 74LS32, Custom:STD_DDW_DIP14, symbol 74xx:74LS32
Connections:
- net GND: now also U3.7 (GND)
- net VCC: now also U3.14 (VCC)
- no-connect marks 17 -> 26
