File: SOUND/soundsch.kicad_sch (KiCad schematic)
At the start: 21 parts, among them J10 DB9_Male, J8 AudioJack3, J9 DB9_Male, P2 CHAN_MIX, U2 W65C22NxP, U25 AY-3-8910

Commit message: sound card working
Parts:
- removed U2: W65C22NxP, Custom:STD_DDW_DIP40, symbol 65xx-library:W65C22NxP
- added U8: 8255, Custom:STD_DDW_DIP40, symbol Interface:8255
- J10, J9: footprint Connector_Dsub:DSUB-9_Pins_Horizontal_P2.77x2.54mm_EdgePinOffset9.40mm -> Connector_Dsub:DSUB-9_Pins_Horizontal_P2.77x2.84mm_EdgePinOffset4.94mm_Housed_MountingHolesOffset4.94mm
- J8: footprint Connector_Audio:Jack_3.5mm_CUI_SJ1-3533NG_Horizontal_CircularHoles -> Custom:ddw_Jack_3.5mm_CUI_SJ1-3525N_Horizontal; symbol Connector:AudioJack3 -> Connector_Audio:AudioJack3
- R10, R11, R12, R13, R14, R8, R9: footprint Resistor_THT:R_Axial_DIN0204_L3.6mm_D1.6mm_P5.08mm_Horizontal -> Custom:STD_DDW_RESISTOR
Connections:
- net A0: now also U8.9 (A0)
- net A1: now also U8.8 (A1)
- net BoardSelect: now also U8.6 (~{CS})
- net D0: now also U8.34 (D0)
- net D1: now also U8.33 (D1)
- net D2: now also U8.32 (D2)
- net D3: now also U8.31 (D3)
- net D4: now also U8.30 (D4)
- net D5: now also U8.29 (D5)
- net D6: now also U8.28 (D6)
- net D7: now also U8.27 (D7)
- net GND: now also J8.S, U8.7 (GND); no longer J8.T
- net RESET: now also U8.35 (RESET); no longer U25.23 (~{RESET})
- net USERA_2: now also U8.16 (PC2)
- net USERA_3: now also U8.17 (PC3)
- net USERA_4: now also U8.13 (PC4)
- net USERB_0: now also U8.18 (PB0)
- net USERB_1: now also U8.19 (PB1)
- net USERB_2: now also U8.20 (PB2)
- net USERB_3: now also U8.21 (PB3)
- net USERB_4: now also U8.22 (PB4)
- net USERB_5: now also U8.23 (PB5)
- net USERB_6: now also U8.24 (PB6)
- net USERB_7: now also U8.25 (PB7)
- net VCC: now also U8.26 (VCC)
- net ~{RESET}: now also U25.23 (~{RESET})
- net at C46.2: now also J8.R; no longer J8.S
- net at C47.2: now also J8.T; no longer J8.R
- new net IOR: U8.5 (~{RD})
- new net IOW: U8.36 (~{WR})
- no-connect marks 19 -> 23
Other:
- moved on the sheet: J8
